File: pcb/airquality.kicad_pcb (KiCad board)
At the start: 2 copper layers, 57 x 47 mm, 7 parts, among them J1 DHT22, J2 PMS7003, U1 ESP32_Wemos

Commit message: update pcb
Parts:
- moved J2 46.3 mm to (147.6, 62.4)
- moved U1 15.9 mm to (177.9, 80.5), turned to 180 degrees
- moved J1 4.99 mm to (188.1, 58.4), turned to 180 degrees
- moved REF** 0.55 mm to (194.5, 52.5)
- moved REF** 0.06 mm to (194.5, 94.5)
- moved REF** 0.06 mm to (142.5, 94.5)
- moved REF** 0.06 mm to (142.5, 52.5)
Routing:
- added copper zone on B.Cu, net GND
- added copper zone on F.Cu, net GND

Commit message: update pcb
Parts:
- moved J2 1.63 mm to (149.0, 61.6)
Changed lines of the file:
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@@
   (general
     (thickness 1.6)
-    (drawings 4)
+    (drawings 8)
     (tracks 0)
     (modules 7)
@@
   )
   (module "Connector_PinHeader_1.00mm:PinHeader_2x05_P1.00mm_Vertical" (layer "F.Cu")
-    (at 147.558 62.4172 180)
+    (at 148.9837 61.6331 180)
     (descr "Through hole straight pin header, 2x05, 1.00mm pitch, double rows")
     (tags "Through hole pin header THT 2x05 1.00mm double row")
@@
     )
     (fp_text value "PMS7003" (at 0.5 5.56) (layer "F.Fab") hide
-      (effects (font (size 1 1) (thickness 0.15)))
-    )
-    (fp_text user "%R" (at 0.5 2 90) (layer "F.Fab")
       (effects (font (size 1 1) (thickness 0.15)))
     )
@@
     (pad "1" np_thru_hole circle (at 0 0) (size 3.2 3.2) (drill 3.2) (layers *.Cu *.Mask))
   )
+  (gr_line (start 144.3194 92.4179) (end 193.3194 92.4179) (layer "F.SilkS") (width 0.12))
+  (gr_line (start 144.3194 54.4179) (end 144.3194 92.4179) (layer "F.SilkS") (width 0.12))
+  (gr_line (start 193.3194 54.4179) (end 193.3194 92.4179) (layer "F.SilkS") (width 0.12))
+  (gr_line (start 144.3194 54.4179) (end 193.3194 54.4179) (layer "F.SilkS") (width 0.12))
   (gr_line (start 197 97) (end 140 97) (layer "Edge.Cuts") (width 0.05))
   (gr_line (start 140 97) (end 140 50) (layer "Edge.Cuts") (width 0.05))

Commit message: update pcb
Parts:
- ESP32 Mini: renamed from U1
- moved PMS7003 2.00 mm to (149.9, 63.4)
- renumbered J1 to DHT22, J2 to PMS7003
Connections:
- ESP32 Mini pad 13: /3V3 -> 5V
- ESP32 Mini pad 14: Net-(U1-Pad14) -> GND
- ESP32 Mini pad 15: Net-(U1-Pad15) -> /RX
- ESP32 Mini pad 16: Net-(U1-Pad16) -> /TX
- ESP32 Mini pad 17: /IO18 -> Net-(U1-Pad17)
- ESP32 Mini pad 20: /RST -> Net-(U1-Pad20)
- ESP32 Mini pad 21: Net-(U1-Pad21) -> /RST
- ESP32 Mini pad 24: Net-(U1-Pad24) -> /IO18
- ESP32 Mini pad 25: /TX -> Net-(U1-Pad25)
- ESP32 Mini pad 26: /RX -> Net-(U1-Pad26)
- ESP32 Mini pad 27: GND -> Net-(U1-Pad27)
- ESP32 Mini pad 28: 5V -> /3V3
Routing:
- net /IO18: track 0.00 -> 54.2 mm
- net /3V3: track 0.00 -> 51.9 mm
- net 5V: track 0.00 -> 46.0 mm
- net /RX: track 0.00 -> 38.6 mm
- net /RST: track 0.00 -> 38.2 mm
- net /TX: track 0.00 -> 34.6 mm
Other:
- board text added: "Air Quality Sensor v0.1 David Davenne 26.05.20"
- board text added: "D"
- board text added: "G"
- board text added: "V+"

Commit message: update pcb
Parts:
- moved PMS7003 1.70 mm to (151.4, 64.3)
Routing:
- net 5V: track 46.0 -> 41.6 mm
- net /RST: track 38.2 -> 37.0 mm
- net /RX: track 38.6 -> 37.9 mm
Other:
- board text added: "Air Quality Sensor v0.1 David Davenne 30.05.20"
- board text added: "JLCJLCJLCJLC"
- board text removed: "Air Quality Sensor v0.1 David Davenne 26.05.20"
